File: templates/atmega2560/atmega2560.sch (KiCad schematic (older format))
At the start: 24 parts, among them J1 INPUT, J2 FTDI, J3 ISP-2560, U1 NCP1117-5V, U2 ATMEGA2560, X1 16MHz 18pF

Commit message: Lots of updates, adjusting templates.
Parts:
- removed S1: RESET, Wickerlib:SW-B3U-1000P, symbol SWITCH-TACTILE-SPST-NO-0.05A-12V
- added S1: RESET, Wickerlib:SWITCH-OMRON-MOMENTARY-SMD-B3U-1000P, symbol SWITCH-MOMENT-SPST-NO-0.05A-12V-SMT-B3U-1000P
- C1, C10, C3, C4, C6, C7, C8, C9, LED1, R2: footprint Wickerlib:0603 -> Wickerlib:RLC-0603-SMD
- C2, C5: footprint Wickerlib:1210 -> Wickerlib:RLC-1210-SMD
- D1, D2, D3: footprint Wickerlib:Diode_SMA -> Wickerlib:DIODE-SMA
- F1: footprint Wickerlib:1812 -> Wickerlib:RLC-1812-SMD
- J2: footprint Wickerlib:Pin_Header_Straight_1x06 -> Wickerlib:CONN-HEADER-STRAIGHT-P2.54MM-1x06
- J3: footprint Wickerlib:Pin_Header_Straight_2x03 -> Wickerlib:CONN-HEADER-STRAIGHT-P2.54MM-2x03
- R1: footprint Wickerlib:0805 -> Wickerlib:RLC-0805-SMD
- U2: footprint TQFP100 -> Wickerlib:TQFP-100-14x14MM-P0.5MM
Other:
- note added: "Analog\nReference\nset to 5V"
- note removed: "Analog\nReference"
Changed lines of the file:
@@
 EESchema Schematic File Version 2
 LIBS:wickerlib
-LIBS:atmega2560-cache
 EELAYER 25 0
 EELAYER END
@@
 F 0 "C2" H 4275 1750 50  0000 L CNN
 F 1 "10uF 25V" H 4275 1650 50  0000 L CNN
-F 2 "Wickerlib:1210" H 4175 1350 50  0001 C CIN
+F 2 "Wickerlib:RLC-1210-SMD" H 4175 1350 50  0001 C CIN
 F 3 "http://www.yuden.co.jp/productdata/catalog/en/mlcc_all_e.pdf" H 4175 1700 5   0001 C CNN
 F 4 "1210" H 4175 1350 50  0001 C CIN "Package"
@@
 F 0 "C5" H 5400 1750 50  0000 L CNN
 F 1 "10uF 25V" H 5400 1650 50  0000 L CNN
-F 2 "Wickerlib:1210" H 5300 1350 50  0001 C CIN
+F 2 "Wickerlib:RLC-1210-SMD" H 5300 1350 50  0001 C CIN
 F 3 "http://www.yuden.co.jp/productdata/catalog/en/mlcc_all_e.pdf" H 5300 1700 5   0001 C CNN
 F 4 "1210" H 5300 1350 50  0001 C CIN "Package"
@@
 F 0 "C3" H 4475 4600 50  0000 L CNN
 F 1 "22pF" H 4475 4500 50  0000 L CNN
-F 2 "Wickerlib:0603" H 4375 4200 50  0001 C CIN
+F 2 "Wickerlib:RLC-0603-SMD" H 4375 4200 50  0001 C CIN
 F 3 "http://www.kemet.com/docfinder?Partnumber=C0603C220F1GACTU" H 4375 4550 5   0001 C CNN
 F 4 "0603" H 4375 4200 50  0001 C CIN "Package"
@@
 F 0 "C4" H 4875 4600 50  0000 L CNN
 F 1 "22pF" H 4875 4500 50  0000 L CNN
-F 2 "Wickerlib:0603" H 4775 4200 50  0001 C CIN
+F 2 "Wickerlib:RLC-0603-SMD" H 4775 4200 50  0001 C CIN
 F 3 "http://www.kemet.com/docfinder?Partnumber=C0603C220F1GACTU" H 4775 4550 5   0001 C CNN
 F 4 "0603" H 4775 4200 50  0001 C CIN "Package"
@@
 F 0 "R1" H 3050 3250 50  0000 L CNN
 F 1 "10K" H 3050 3150 50  0000 L CNN
-F 2 "Wickerlib:0805" H 2975 2850 50  0001 C CIN
+F 2 "Wickerlib:RLC-0805-SMD" H 2975 2850 50  0001 C CIN
 F 3 "http://www.yageo.com/NewPortal/yageodocoutput?fileName=/pdf/R-Chip/PYu-RC_Group_51_RoHS_L_3.pdf" H 2975 3200 5   0001 C CNN
 F 4 "0805" H 2975 2850 50  0001 C CIN "Package"
@@
 F 0 "D1" H 2825 1800 50  0000 L CNN
 F 1 "14V" H 2825 1700 50  0000 L CNN
-F 2 "Wickerlib:Diode_SMA" H 2750 1400 50  0001 C CIN
+F 2 "Wickerlib:DIODE-SMA" H 2750 1400 50  0001 C CIN
 F 3 "http://www.ti.com/lit/ds/symlink/tpd3e001.pdf" V 2750 1750 5   0001 C CNN
 F 4 "SMA" H 2750 1400 50  0001 C CIN "Package"
@@
 F 0 "F1" V 3400 1450 50  0000 L CNN
 F 1 "1.1A 25V" V 3550 1350 50  0000 L CNN
-F 2 "Wickerlib:1812" H 3475 1150 50  0001 C CIN
+F 2 "Wickerlib:RLC-1812-SMD" H 3475 1150 50  0001 C CIN
 F 3 "http://www.bourns.com/docs/Product-Datasheets/mfmsmf.pdf" H 3475 1500 5   0001 C CNN
 F 4 "1812" H 3475 1150 50  0001 C CIN "Package"
@@
 U 1 1 573232D9
 P 3025 1500
-F 0 "D2" H 2975 1400 50  0000 L CNN
-F 1 "20V 1A" H 2900 1600 50  0000 L CNN
-F 2 "Wickerlib:Diode_SMA" H 3025 1150 50  0001 C CIN
+F 0 "D2" V 2925 1450 50  0000 L CNN
+F 1 "20V 1A" V 3125 1375 50  0000 L CNN
+F 2 "Wickerlib:DIODE-SMA" H 3025 1150 50  0001 C CIN
 F 3 "http://www.vishay.com/docs/88746/ss12.pdf" H 3025 1500 5   0001 C CNN
 F 4 "UNDEFINED" H 3025 1150 50  0001 C CIN "Package"
@@
 F 10 "Not Verified" H 3025 1150 50  0001 C CIN "Verified"
 	1    3025 1500
-	-1   0    0    1
+	0    1    1    0
 $EndComp
 $Comp
@@
 F 0 "C7" H 6900 2950 50  0000 L CNN
 F 1 "100nF" H 6900 2850 50  0000 L CNN
-F 2 "Wickerlib:0603" H 6800 2550 50  0001 C CIN
+F 2 "Wickerlib:RLC-0603-SMD" H 6800 2550 50  0001 C CIN
 F 3 "http://search.murata.co.jp/Ceramy/image/img/A01X/partnumbering_e_01.pdf" H 6800 2900 5   0001 C CNN
 F 4 "0603" H 6800 2550 50  0001 C CIN "Package"
@@
 F 0 "C8" H 7325 2950 50  0000 L CNN
 F 1 "100nF" H 7325 2850 50  0000 L CNN
-F 2 "Wickerlib:0603" H 7225 2550 50  0001 C CIN
+F 2 "Wickerlib:RLC-0603-SMD" H 7225 2550 50  0001 C CIN
 F 3 "http://search.murata.co.jp/Ceramy/image/img/A01X/partnumbering_e_01.pdf" H 7225 2900 5   0001 C CNN
 F 4 "0603" H 7225 2550 50  0001 C CIN "Package"
@@
 F 0 "C9" H 7775 2950 50  0000 L CNN
 F 1 "100nF" H 7775 2850 50  0000 L CNN
-F 2 "Wickerlib:0603" H 7675 2550 50  0001 C CIN
+F 2 "Wickerlib:RLC-0603-SMD" H 7675 2550 50  0001 C CIN
 F 3 "http://search.murata.co.jp/Ceramy/image/img/A01X/partnumbering_e_01.pdf" H 7675 2900 5   0001 C CNN
 F 4 "0603" H 7675 2550 50  0001 C CIN "Package"
@@
 $EndComp
 $Comp
-L SWITCH-TACTILE-SPST-NO-0.05A-12V S1
-U 1 1 572E9065
-P 2725 3400
-F 0 "S1" H 2550 3500 50  0000 L CNN
-F 1 "RESET" H 2525 3325 50  0000 L CNN
-F 2 "Wickerlib:SW-B3U-1000P" H 2725 3050 50  0001 C CIN
-F 3 "http://www.omron.com/ecb/products/pdf/en-b3u.pdf" H 2725 3400 5   0001 C CNN
-F 4 "SW-B3F-10XX" H 2725 3050 50  0001 C CIN "Package"
-F 5 "Omron" H 2725 3050 50  0001 C CIN "MF_Name"
-F 6 "B3U-1000P" H 2725 3050 50  0001 C CIN "MF_PN"
-F 7 "Digikey" H 2725 3050 50  0001 C CIN "S1_Name"
-F 8 "SW1020CT-ND" H 2725 3050 50  0001 C CIN "S1_PN"
-F 9 "SWITCH TACTILE SPST-NO 0.05A 12V" H 2725 3050 50  0001 C CIN "Description"
-F 10 "Not Verified" H 2725 3050 50  0001 C CIN "Verified"
-	1    2725 3400
-	1    0    0    -1
-$EndComp
-$Comp
 L HEADER-MALE-6POS-TH-2x3-P0.1IN J3
 U 1 1 5745627C
@@
 F 0 "J3" H 4025 3500 50  0000 L CNN
 F 1 "ISP-2560" H 3925 3100 50  0000 L CNN
-F 2 "Wickerlib:Pin_Header_Straight_2x03" H 4100 2950 50  0001 C CIN
+F 2 "Wickerlib:CONN-HEADER-STRAIGHT-P2.54MM-2x03" H 4100 2950 50  0001 C CIN
 F 3 "http://cdn.harwin.com/pdfs/60page147.pdf" H 4100 3300 5   0001 C CNN
 F 4 "UNDEFINED" H 4100 2950 50  0001 C CIN "Package"
@@
 F 0 "C1" H 3575 4250 50  0000 L CNN
 F 1 "100nF" H 3575 4150 50  0000 L CNN
-F 2 "Wickerlib:0603" H 3475 3850 50  0001 C CIN
+F 2 "Wickerlib:RLC-0603-SMD" H 3475 3850 50  0001 C CIN
 F 3 "http://search.murata.co.jp/Ceramy/image/img/A01X/partnumbering_e_01.pdf" H 3475 4200 5   0001 C CNN
 F 4 "0603" H 3475 3850 50  0001 C CIN "Package"
@@
 F 0 "J2" H 2150 4950 50  0000 L CNN
 F 1 "FTDI" H 2125 4225 50  0001 L CNN
-F 2 "Wickerlib:Pin_Header_Straight_1x06" H 2175 4250 50  0001 C CIN
+F 2 "Wickerlib:CONN-HEADER-STRAIGHT-P2.54MM-1x06" H 2175 4250 50  0001 C CIN
 F 3 "https://cdn.harwin.com/pdfs/60page140.pdf" H 2175 4600 5   0001 C CNN
 F 4 "Pin_Header_Straight_1x06" H 2175 4250 50  0001 C CIN "Package"
@@
 U 1 1 574C79CC
 P 5800 1500
-F 0 "D3" H 5750 1400 50  0000 L CNN
-F 1 "20V 1A" H 5675 1600 50  0000 L CNN
-F 2 "Wickerlib:Diode_SMA" H 5800 1150 50  0001 C CIN
+F 0 "D3" V 5700 1450 50  0000 L CNN
+F 1 "20V 1A" V 5900 1350 50  0000 L CNN
+F 2 "Wickerlib:DIODE-SMA" H 5800 1150 50  0001 C CIN
 F 3 "http://www.vishay.com/docs/88746/ss12.pdf" H 5800 1500 5   0001 C CNN
 F 4 "UNDEFINED" H 5800 1150 50  0001 C CIN "Package"
@@
 F 10 "Not Verified" H 5800 1150 50  0001 C CIN "Verified"
 	1    5800 1500
-	-1   0    0    1
+	0    1    1    0
 $EndComp
 NoConn ~ 2375 4750
@@
 F 0 "R2" H 8000 5700 50  0000 L CNN
 F 1 "1K" H 8000 5600 50  0000 L CNN
-F 2 "Wickerlib:0603" H 7950 5300 50  0001 C CIN
+F 2 "Wickerlib:RLC-0603-SMD" H 7950 5300 50  0001 C CIN
 F 3 "http://media.digikey.com/pdf/Data%20Sheets/Samsung%20PDFs/RC_Series_ds.pdf" H 7950 5650 5   0001 C CNN
 F 4 "0603" H 7950 5300 50  0001 C CIN "Package"
@@
 F 0 "LED1" H 8000 5975 50  0000 L CNN
 F 1 "AMBER" H 8000 5875 50  0000 L CNN
-F 2 "Wickerlib:0603" H 7950 5575 50  0001 C CIN
+F 2 "Wickerlib:RLC-0603-SMD" H 7950 5575 50  0001 C CIN
 F 3 "http://media.digikey.com/pdf/Data%20Sheets/Osram%20PDFs/LSLALOLY_296.pdf" V 7950 5925 5   0001 C CNN
 F 4 "0603" H 7950 5575 50  0001 C CIN "Package"
@@
 $EndComp
 Text Notes 5300 2575 0    60   ~ 0
-   Analog\nReference
+   Analog\nReference\nset to 5V
 $Comp
 L GND #PWR022
@@
 F 0 "C6" H 5450 2950 50  0000 L CNN
 F 1 "100nF" H 5450 2850 50  0000 L CNN
-F 2 "Wickerlib:0603" H 5350 2550 50  0001 C CIN
+F 2 "Wickerlib:RLC-0603-SMD" H 5350 2550 50  0001 C CIN
 F 3 "http://search.murata.co.jp/Ceramy/image/img/A01X/partnumbering_e_01.pdf" H 5350 2900 5   0001 C CNN
 F 4 "0603" H 5350 2550 50  0001 C CIN "Package"
@@
 F 0 "C10" H 8250 2950 50  0000 L CNN
 F 1 "100nF" H 8250 2850 50  0000 L CNN
-F 2 "Wickerlib:0603" H 8150 2550 50  0001 C CIN
+F 2 "Wickerlib:RLC-0603-SMD" H 8150 2550 50  0001 C CIN
 F 3 "http://search.murata.co.jp/Ceramy/image/img/A01X/partnumbering_e_01.pdf" H 8150 2900 5   0001 C CNN
 F 4 "0603" H 8150 2550 50  0001 C CIN "Package"
@@
 F 0 "U2" H 5325 8925 50  0000 L BNN
 F 1 "ATMEGA2560" H 7150 6275 50  0000 L BNN
-F 2 "TQFP100" H 6525 6275 50  0001 C CIN
+F 2 "Wickerlib:TQFP-100-14x14MM-P0.5MM" H 6525 6275 50  0001 C CIN
 F 3 "http://www.atmel.com/Images/Atmel-2549-8-bit-AVR-Microcontroller-ATmega640-1280-1281-2560-2561_Summary.pdf" H 6075 9375 50  0001 C CNN
 F 4 "TQFP100" H 6075 9425 50  0001 C CIN "Package"
@@
 	1    0    0    -1
 $EndComp
+$Comp
+L SWITCH-MOMENT-SPST-NO-0.05A-12V-SMT-B3U-1000P S1
+U 1 1 599247AF
+P 2725 3400
+F 0 "S1" H 2625 3550 50  0000 L CNN
+F 1 "RESET" H 2525 3325 50  0000 L CNN
+F 2 "Wickerlib:SWITCH-OMRON-MOMENTARY-SMD-B3U-1000P" H 2725 3050 50  0001 C CIN
+F 3 "http://www.omron.com/ecb/products/pdf/en-b3u.pdf" H 2725 3400 5   0001 C CNN
+F 4 "SWITCH TACTILE SPST-NO 0.05A 12V" H 2725 3050 50  0001 C CIN "Description"
+F 5 "Omron" H 2725 3050 50  0001 C CIN "MF_Name"
+F 6 "B3U-1000P" H 2725 3050 50  0001 C CIN "MF_PN"
+F 7 "Digikey" H 2725 3050 50  0001 C CIN "S1_Name"
+F 8 "SW1020CT-ND" H 2725 3050 50  0001 C CIN "S1_PN"
+	1    2725 3400
+	1    0    0    -1
+$EndComp

Commit message: Move template cleanup.
Parts:
- C1, C10, C3, C4, C6, C7, C8, C9, LED1, R2: Package 0603 -> (none); Verified Not Verified -> (none)
- C2, C5: Package 1210 -> (none); Verified Not Verified -> (none)
- D1: Package SMA -> (none); Verified Not Verified -> (none)
- D2, D3, J3: Package UNDEFINED -> (none); Verified Not Verified -> (none)
- F1: Package 1812 -> (none); Verified Not Verified -> (none)
- J1: footprint Wickerlib:OSTVN02A150 -> Wickerlib:CONN-ONSHORE-SCREW-GREEN-2PIN-TH; Package OSTVN02A150 -> (none); Verified Not Verified -> (none)
- J2: Package Pin_Header_Straight_1x06 -> (none); Verified Not Verified -> (none)
- R1: Package 0805 -> (none); Verified Not Verified -> (none)
- U1: Package DPAK -> (none); Verified Not Verified -> (none)
- U2: Package TQFP100 -> (none); Verified Not Verified -> (none)
- X1: Package CRYSTAL-CTS-4SMD -> (none); Verified Not Verified -> (none)
