File: templates/atmega2560/atmega2560.kicad_pcb (KiCad board)
At the start: 2 copper layers, 0 parts

Commit message: Add fab notes to Dwgs.User
Other:
- board text added: "FABRICATION NOTES 1. THIS IS A 2 LAYER BOARD. 2. EXTERNAL LAYERS SHALL HAVE 1 OZ COPPER. 3. MATERIAL: FR4 AND 0.062 INCH +/- 10% THICK. 4. BOARDS SHALL BE ROHS COMPLIANT. 5. MANUFACTURE IN ACCORDANCE WITH IPC-6012 CLASS 2 6. MASK: BOTH SIDES OF THE BOARD SHALL HAVE SOLDER MASK (ANY COLOR) OVER BARE COPPER. 7. SILK: BOTH SIDES OF THE BOARD SHALL HAVE WHITE SILKSCREEN. DO NOT PLACE SILK OVER BARE C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"
Changed lines of the file:
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@@
-(kicad_pcb (version 4) (host pcbnew 4.0.5-e0-6337~49~ubuntu16.04.1)
+(kicad_pcb (version 4) (host pcbnew 4.0.7-e2-6376~58~ubuntu16.04.1)
   (general
-    (links 59)
-    (no_connects 41)
+    (links 0)
+    (no_connects 0)
     (area 0 0 0 0)
     (thickness 1.6)
-    (drawings 0)
+    (drawings 1)
     (tracks 0)
     (zones 0)
@@
     (uvia_dia 0.6858)
     (uvia_drill 0.3302)
-    (add_net +12V)
-    (add_net +5V)
-    (add_net /FTDI_RESET)
-    (add_net /FTDI_RXIN)
-    (add_net /FTDI_TXOUT)
-    (add_net /MISO2)
-    (add_net /MOSI2)
-    (add_net /SCK2)
-    (add_net /VIN)
-    (add_net /~RESET2)
-    (add_net GND)
-    (add_net "Net-(C3-Pad1)")
-    (add_net "Net-(C4-Pad1)")
-    (add_net "Net-(C5-Pad1)")
-    (add_net "Net-(D2-Pad1)")
-    (add_net "Net-(LED1-Pad2)")
-    (add_net "Net-(R2-Pad1)")
+  )
+  (gr_text "FABRICATION NOTES\n\n1. THIS IS A 2 LAYER BOARD. \n2. EXTERNAL LAYERS SHALL HAVE 1 OZ COPPER.\n3. MATERIAL: FR4 AND 0.062 INCH +/- 10% THICK.\n4. BOARDS SHALL BE ROHS COMPLIANT. \n5. MANUFACTURE IN ACCORDANCE WITH IPC-6012 CLASS 2\n6. MASK: BOTH SIDES OF THE BOARD SHALL HAVE \n   SOLDER MASK (ANY COLOR) OVER BARE COPPER. \n7. SILK: BOTH SIDES OF THE BOARD SHALL HAVE \n   WHITE SILKSCREEN. DO NOT PLACE SILK OVER BARE COPPER.\n8. FINISH: ENIG.\n9. MINIMUM TRACE WIDTH - 0.006 INCH.\n   MINIMUM SPACE - 0.006 INCH.\n   MINIMUM HOLE DIA - 0.013 INCH. \n10. MAX HOLE PLACEMENT TOLERANCE OF +/- 0.003 INCH.\n11. MAX HOLE DIAMETER TOLERANCE OF +/- 0.003 INCH AFTER PLATING." (at 113.5888 95.9104) (layer Dwgs.User)
+    (effects (font (size 2.54 2.54) (thickness 0.254)) (justify left))
   )
 )
