File: templates/teensy-3.2/teensy-3.2.sch (KiCad schematic (older format))
At the start: 1 part, among them J1 TEENSY3.2-72MHz

Commit message: Moved wickerbox templates out. Teensy is messed up.
Parts:
- J1: footprint Wickerlib:TEENSY-3.2 -> Wickerlib:TEENSY-3.2-NOSILK; Package UNDEFINED -> (none); Verified Not Verified -> (none)
Changed lines of the file:
@@
 EESchema Schematic File Version 2
-LIBS:teensy-3.2-cache
 LIBS:wickerlib
 EELAYER 25 0
@@
 F 0 "J1" H 2500 5700 50  0000 L CNN
 F 1 "TEENSY3.2-72MHz" H 2500 2050 50  0000 L CNN
-F 2 "Wickerlib:TEENSY-3.2" V 2450 5000 50  0001 C CIN
+F 2 "Wickerlib:TEENSY-3.2-NOSILK" V 2450 5000 50  0001 C CIN
 F 3 "https://www.pjrc.com/teensy/" H 2950 4500 5   0001 C CNN
-F 4 "UNDEFINED" V 2450 5000 50  0001 C CIN "Package"
-F 5 "PJRC" V 2450 5000 50  0001 C CIN "MF_Name"
-F 6 "TEENSY3.2" V 2450 5000 50  0001 C CIN "MF_PN"
-F 7 "PJRC" V 2450 5000 50  0001 C CIN "S1_Name"
-F 8 "TEENSY3.2" V 2450 5000 50  0001 C CIN "S1_PN"
-F 9 "TEENSY 3.2 32BIT 72MHZ" V 2450 5000 50  0001 C CIN "Description"
-F 10 "Not Verified" V 2450 5000 50  0001 C CIN "Verified"
+F 4 "PJRC" V 2450 5000 50  0001 C CIN "MF_Name"
+F 5 "TEENSY3.2" V 2450 5000 50  0001 C CIN "MF_PN"
+F 6 "PJRC" V 2450 5000 50  0001 C CIN "S1_Name"
+F 7 "TEENSY3.2" V 2450 5000 50  0001 C CIN "S1_PN"
+F 8 "TEENSY 3.2 32BIT 72MHZ" V 2450 5000 50  0001 C CIN "Description"
 	1    2700 3850
 	1    0    0    -1
