File: templates/atmega328/atmega328.kicad_pcb (KiCad board)
At the start: 2 copper layers, 0 parts

Commit message: Lots of updates, adjusting templates.
Other:
- rule trace_clearance: 0.254 -> 0.2
Changed lines of the file:
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@@
-(kicad_pcb (version 4) (host pcbnew 4.0.4+e1-6308~48~ubuntu14.04.1-stable)
+(kicad_pcb (version 4) (host pcbnew 4.0.5-e0-6337~49~ubuntu16.04.1)
   (general
     (links 0)
@@
     (0 F.Cu signal)
     (31 B.Cu signal)
-    (32 B.Adhes user)
-    (33 F.Adhes user)
     (34 B.Paste user)
     (35 F.Paste user)
@@
     (39 F.Mask user)
     (40 Dwgs.User user)
-    (41 Cmts.User user)
-    (42 Eco1.User user)
-    (43 Eco2.User user)
     (44 Edge.Cuts user)
-    (45 Margin user)
-    (46 B.CrtYd user)
-    (47 F.CrtYd user)
-    (48 B.Fab user)
-    (49 F.Fab user)
-  )
-  (layers
-    (0 F.Cu signal)
-    (31 B.Cu signal)
-    (34 B.Paste user)
-    (35 F.Paste user)
-    (36 B.SilkS user)
-    (37 F.SilkS user)
-    (38 B.Mask user)
-    (39 F.Mask user)
-    (44 Edge.Cuts user)
-    (46 B.CrtYd user)
-    (47 F.CrtYd user)
     (48 B.Fab user)
     (49 F.Fab user)
   )
   (setup
-    (last_trace_width 0.254)
+    (last_trace_width 0.25)
     (user_trace_width 0.1524)
     (user_trace_width 0.254)
@@
     (user_trace_width 0.762)
     (user_trace_width 1.27)
-    (trace_clearance 0.254)
+    (trace_clearance 0.2)
     (zone_clearance 0.508)
     (zone_45_only no)
@@
     (segment_width 0.1524)
     (edge_width 0.1524)
-    (via_size 0.6858)
-    (via_drill 0.3302)
+    (via_size 0.6)
+    (via_drill 0.4)
     (via_min_size 0.6858)
     (via_min_drill 0.3302)
@@
     (user_via 0.762 0.4064)
     (user_via 0.8636 0.508)
-    (uvia_size 0.6858)
-    (uvia_drill 0.3302)
+    (uvia_size 0.3)
+    (uvia_drill 0.1)
     (uvias_allowed no)
     (uvia_min_size 0)

Commit message: Add fab notes to Dwgs.User
Other:
- board text added: "FABRICATION NOTES 1. THIS IS A 2 LAYER BOARD. 2. EXTERNAL LAYERS SHALL HAVE 1 OZ COPPER. 3. MATERIAL: FR4 AND 0.062 INCH +/- 10% THICK. 4. BOARDS SHALL BE ROHS COMPLIANT. 5. MANUFACTURE IN ACCORDANCE WITH IPC-6012 CLASS 2 6. MASK: BOTH SIDES OF THE BOARD SHALL HAVE SOLDER MASK (ANY COLOR) OVER BARE COPPER. 7. SILK: BOTH SIDES OF THE BOARD SHALL HAVE WHITE SILKSCREEN. DO NOT PLACE SILK OVER BARE C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"
Changed lines of the file:
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@@
-(kicad_pcb (version 4) (host pcbnew 4.0.5-e0-6337~49~ubuntu16.04.1)
+(kicad_pcb (version 4) (host pcbnew 4.0.7-e2-6376~58~ubuntu16.04.1)
   (general
-    (links 73)
-    (no_connects 56)
+    (links 0)
+    (no_connects 0)
     (area 0 0 0 0)
     (thickness 1.6)
-    (drawings 0)
+    (drawings 1)
     (tracks 0)
     (zones 0)
@@
     (uvia_dia 0.3)
     (uvia_drill 0.1)
-    (add_net +12V)
-    (add_net +5V)
-    (add_net /A0)
-    (add_net /A1)
-    (add_net /A2)
-    (add_net /A3)
-    (add_net /A4)
-    (add_net /A5)
-    (add_net "/A6(*)")
-    (add_net "/A7(*)")
-    (add_net /D0)
-    (add_net /D1)
-    (add_net /D10)
-    (add_net /D11)
-    (add_net /D12)
-    (add_net /D13)
-    (add_net /D2)
-    (add_net /D3)
-    (add_net /D4)
-    (add_net /D5)
-    (add_net /D6)
-    (add_net /D7)
-    (add_net /D8)
-    (add_net /D9)
-    (add_net /FTDI_RESET)
-    (add_net /VIN)
-    (add_net /~RESET)
-    (add_net GND)
-    (add_net "Net-(C3-Pad1)")
-    (add_net "Net-(C4-Pad1)")
-    (add_net "Net-(C6-Pad1)")
-    (add_net "Net-(D2-Pad1)")
-    (add_net "Net-(LED1-Pad2)")
+  )
+  (gr_text "FABRICATION NOTES\n\n1. THIS IS A 2 LAYER BOARD. \n2. EXTERNAL LAYERS SHALL HAVE 1 OZ COPPER.\n3. MATERIAL: FR4 AND 0.062 INCH +/- 10% THICK.\n4. BOARDS SHALL BE ROHS COMPLIANT. \n5. MANUFACTURE IN ACCORDANCE WITH IPC-6012 CLASS 2\n6. MASK: BOTH SIDES OF THE BOARD SHALL HAVE \n   SOLDER MASK (ANY COLOR) OVER BARE COPPER. \n7. SILK: BOTH SIDES OF THE BOARD SHALL HAVE \n   WHITE SILKSCREEN. DO NOT PLACE SILK OVER BARE COPPER.\n8. FINISH: ENIG.\n9. MINIMUM TRACE WIDTH - 0.006 INCH.\n   MINIMUM SPACE - 0.006 INCH.\n   MINIMUM HOLE DIA - 0.013 INCH. \n10. MAX HOLE PLACEMENT TOLERANCE OF +/- 0.003 INCH.\n11. MAX HOLE DIAMETER TOLERANCE OF +/- 0.003 INCH AFTER PLATING." (at 115.2144 91.9988) (layer Dwgs.User)
+    (effects (font (size 2.54 2.54) (thickness 0.254)) (justify left))
   )
 )
