File: templates/oshpark-2layer/oshpark-2layer.kicad_pcb (KiCad board)
At the start: 2 copper layers, 0 parts

Commit message: Add fab notes to Dwgs.User
Other:
- board text added: "FABRICATION NOTES 1. THIS IS A 2 LAYER BOARD. 2. EXTERNAL LAYERS SHALL HAVE 1 OZ COPPER. 3. MATERIAL: FR4 AND 0.062 INCH +/- 10% THICK. 4. BOARDS SHALL BE ROHS COMPLIANT. 5. MANUFACTURE IN ACCORDANCE WITH IPC-6012 CLASS 2 6. MASK: BOTH SIDES OF THE BOARD SHALL HAVE SOLDER MASK (ANY COLOR) OVER BARE COPPER. 7. SILK: BOTH SIDES OF THE BOARD SHALL HAVE WHITE SILKSCREEN. DO NOT PLACE SILK OVER BARE C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"
Changed lines of the file:
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@@
-(kicad_pcb (version 4) (host pcbnew 4.0.1-3.201512221402+6198~38~ubuntu14.04.1-stable)
+(kicad_pcb (version 4) (host pcbnew 4.0.7-e2-6376~58~ubuntu16.04.1)
   (general
     (links 0)
@@
     (area 104.572999 74.854999 178.510001 123.265001)
     (thickness 1.6)
-    (drawings 17)
+    (drawings 1)
     (tracks 0)
     (zones 0)
@@
     (38 B.Mask user)
     (39 F.Mask user)
+    (40 Dwgs.User user)
     (44 Edge.Cuts user)
     (46 B.CrtYd user)
@@
     (uvia_drill 0.3302)
   )
-  (gr_circle (center 117.348 76.962) (end 118.618 76.962) (layer Dwgs.User) (width 0.15))
-  (gr_line (start 114.427 78.994) (end 114.427 74.93) (angle 90) (layer Dwgs.User) (width 0.15))
-  (gr_line (start 120.269 78.994) (end 114.427 78.994) (angle 90) (layer Dwgs.User) (width 0.15))
-  (gr_line (start 120.269 74.93) (end 120.269 78.994) (angle 90) (layer Dwgs.User) (width 0.15))
-  (gr_line (start 114.427 74.93) (end 120.269 74.93) (angle 90) (layer Dwgs.User) (width 0.15))
-  (gr_line (start 120.523 93.98) (end 104.648 93.98) (angle 90) (layer Dwgs.User) (width 0.15))
-  (gr_line (start 173.355 102.235) (end 173.355 94.615) (angle 90) (layer Dwgs.User) (width 0.15))
-  (gr_line (start 178.435 102.235) (end 173.355 102.235) (angle 90) (layer Dwgs.User) (width 0.15))
-  (gr_line (start 178.435 94.615) (end 178.435 102.235) (angle 90) (layer Dwgs.User) (width 0.15))
-  (gr_line (start 173.355 94.615) (end 178.435 94.615) (angle 90) (layer Dwgs.User) (width 0.15))
-  (gr_line (start 109.093 123.19) (end 109.093 114.3) (angle 90) (layer Dwgs.User) (width 0.15))
-  (gr_line (start 122.428 123.19) (end 109.093 123.19) (angle 90) (layer Dwgs.User) (width 0.15))
-  (gr_line (start 122.428 114.3) (end 122.428 123.19) (angle 90) (layer Dwgs.User) (width 0.15))
-  (gr_line (start 109.093 114.3) (end 122.428 114.3) (angle 90) (layer Dwgs.User) (width 0.15))
-  (gr_line (start 104.648 93.98) (end 104.648 82.55) (angle 90) (layer Dwgs.User) (width 0.15))
-  (gr_line (start 120.523 82.55) (end 120.523 93.98) (angle 90) (layer Dwgs.User) (width 0.15))
-  (gr_line (start 104.648 82.55) (end 120.523 82.55) (angle 90) (layer Dwgs.User) (width 0.15))
+  (gr_text "FABRICATION NOTES\n\n1. THIS IS A 2 LAYER BOARD. \n2. EXTERNAL LAYERS SHALL HAVE 1 OZ COPPER.\n3. MATERIAL: FR4 AND 0.062 INCH +/- 10% THICK.\n4. BOARDS SHALL BE ROHS COMPLIANT. \n5. MANUFACTURE IN ACCORDANCE WITH IPC-6012 CLASS 2\n6. MASK: BOTH SIDES OF THE BOARD SHALL HAVE \n   SOLDER MASK (ANY COLOR) OVER BARE COPPER. \n7. SILK: BOTH SIDES OF THE BOARD SHALL HAVE \n   WHITE SILKSCREEN. DO NOT PLACE SILK OVER BARE COPPER.\n8. FINISH: ENIG.\n9. MINIMUM TRACE WIDTH - 0.006 INCH.\n   MINIMUM SPACE - 0.006 INCH.\n   MINIMUM HOLE DIA - 0.013 INCH. \n10. MAX HOLE PLACEMENT TOLERANCE OF +/- 0.003 INCH.\n11. MAX HOLE DIAMETER TOLERANCE OF +/- 0.003 INCH AFTER PLATING." (at 113.4872 93.2688) (layer Dwgs.User)
+    (effects (font (size 2.54 2.54) (thickness 0.254)) (justify left))
+  )
 )
